Commit message: 初步搭建强化学习代码

File: m4lp.urdf (robot description, URDF)
Before this commit: robot M4LP, 25 links, 24 joints
Joints:
- joint FL_wheel_joint: axis (none) -> 1 0 0; limit (none) -> effort=20 velocity=50; origin xyz=0 0 0 rpy=0 0 0 -> xyz=0 0 -0.125 rpy=0 0 0; type fixed -> continuous
- joint FR_wheel_joint: axis (none) -> 1 0 0; limit (none) -> effort=20 velocity=50; origin xyz=0 0 0 rpy=0 0 0 -> xyz=0 0 -0.125 rpy=0 0 0; type fixed -> continuous
- joint RL_wheel_joint: axis (none) -> 1 0 0; limit (none) -> effort=20 velocity=50; origin xyz=0 0 0 rpy=0 0 0 -> xyz=0 0 -0.125 rpy=0 0 0; type fixed -> continuous
- joint RR_wheel_joint: axis (none) -> 1 0 0; limit (none) -> effort=20 velocity=50; origin xyz=0 0 0 rpy=0 0 0 -> xyz=0 0 -0.125 rpy=0 0 0; type fixed -> continuous

Commit message: Update m4lp.urdf

File: m4lp.urdf (robot description, URDF)
Before this commit: robot M4LP, 25 links, 24 joints
Joints:
- joint FL_wheel_joint: axis 1 0 0 -> 0 0 1; origin xyz=0 0 -0.125 rpy=0 0 0 -> xyz=0 0 -0.25 rpy=1.57 0 0
- joint FR_wheel_joint: axis 1 0 0 -> 0 0 1; origin xyz=0 0 -0.125 rpy=0 0 0 -> xyz=0 0 -0.25 rpy=1.57 0 0
- joint RL_wheel_joint: axis 1 0 0 -> 0 0 1; origin xyz=0 0 -0.125 rpy=0 0 0 -> xyz=0 0 -0.25 rpy=1.57 0 0
- joint RR_wheel_joint: axis 1 0 0 -> 0 0 1; origin xyz=0 0 -0.125 rpy=0 0 0 -> xyz=0 0 -0.25 rpy=1.57 0 0

Commit message: 基础前后及上下控制

File: m4lp.urdf (robot description, URDF)
Before this commit: robot M4LP, 25 links, 24 joints
Links:
- link FL_hip: mass 0.1 -> 0.3
- link FL_shank: mass 0.12 -> 0.6
- link FL_thigh: mass 0.15 -> 0.8
- link FL_wheel: mass 0.08 -> 0.4
- link FR_hip: mass 0.1 -> 0.3
- link FR_shank: mass 0.12 -> 0.6
- link FR_thigh: mass 0.15 -> 0.8
- link FR_wheel: mass 0.08 -> 0.4
- link RL_hip: mass 0.1 -> 0.3
- link RL_shank: mass 0.12 -> 0.6
- link RL_thigh: mass 0.15 -> 0.8
- link RL_wheel: mass 0.08 -> 0.4
- link RR_hip: mass 0.1 -> 0.3
- link RR_shank: mass 0.12 -> 0.6
- link RR_thigh: mass 0.15 -> 0.8
- link RR_wheel: mass 0.08 -> 0.4
- link base: mass 2.0 -> 8.0

Commit message: 增加陀螺仪

File: m4lp.urdf (robot description, URDF)
Before this commit: robot M4LP, 25 links, 24 joints
Links:
- added link gyroscope, mass 0.01
Joints:
- added joint gyroscope_joint: type fixed, parent base, child gyroscope, origin xyz=0 0 0 rpy=0 0 0

Commit message: xbox手柄版重构

File: m4lp.urdf (robot description, URDF)
Before this commit: robot M4LP, 26 links, 25 joints
Links:
- link FL_hip: mass 0.3 -> 0.05
- link FL_shank: mass 0.6 -> 0.1
- link FL_thigh: mass 0.8 -> 0.15
- link FL_wheel: mass 0.4 -> 0.08
- link FR_hip: mass 0.3 -> 0.05
- link FR_shank: mass 0.6 -> 0.1
- link FR_thigh: mass 0.8 -> 0.15
- link FR_wheel: mass 0.4 -> 0.08
- link RL_hip: mass 0.3 -> 0.05
- link RL_shank: mass 0.6 -> 0.1
- link RL_thigh: mass 0.8 -> 0.15
- link RL_wheel: mass 0.4 -> 0.08
- link RR_hip: mass 0.3 -> 0.05
- link RR_shank: mass 0.6 -> 0.1
- link RR_thigh: mass 0.8 -> 0.15
- link RR_wheel: mass 0.4 -> 0.08
- link base: mass 8.0 -> 10.0
